Commit message: Integrate unified robot API and profile-driven camera recording

File: adapters/robots/openarmx/urdf/openarmx_robot.urdf (robot description, URDF)
Before this commit: robot openarmx, 30 links, 29 joints
Links:
- added link L_Link7_XJ_Link, mass 0.0389014964910646; collision mesh filename=../meshes/cameras/L_Link7_XJ_Link.STL; visual mesh filename=../meshes/cameras/L_Link7_XJ_Link.STL
- added link R_LINK7_XJ_Link, mass 0.0389014964910647; collision mesh filename=../meshes/cameras/R_LINK7_XJ_Link.STL; visual mesh filename=../meshes/cameras/R_LINK7_XJ_Link.STL
- added link XJZJ_Link, mass 0.0533057089381443; collision mesh filename=../meshes/cameras/XJZJ_Link.STL; visual mesh filename=../meshes/cameras/XJZJ_Link.STL
- added link XJ_Link, mass 0.0456898574293222; collision mesh filename=../meshes/cameras/XJ_Link.STL; visual mesh filename=../meshes/cameras/XJ_Link.STL
Joints:
- added joint L_Link7_XJ_joint: type fixed, parent openarmx_left_link7, child L_Link7_XJ_Link, origin xyz=0.10811 0 0.082659 rpy=2.618 -3.1416 -1.5708, axis 0 0 0
- added joint R_LINK7_XJ: type fixed, parent openarmx_right_link7, child R_LINK7_XJ_Link, origin xyz=0.108111848164622 0 0.0816585089852266 rpy=0 -0.523598775598298 0, axis 0 0 0
- added joint XJ: type fixed, parent XJZJ_Link, child XJ_Link, origin xyz=0.0484847918575208 0 0.101257907919113 rpy=-3.14159265358979 0.698131700797709 3.14159265358979, axis 0 0 0
- added joint XJZJ: type fixed, parent openarmx_body_link0, child XJZJ_Link, origin xyz=0.00321 0 0.81297 rpy=0 0 0, axis 0 0 0
